File: hardware/pcb-v1/meteohubsensor-v1.kicad_pcb (KiCad board)
At the start: 2 copper layers, 66 x 50 mm, 18 parts, among them J1 BAT, J2 BMP280, J3 DHT22, J4 ANEMO, J5 PLUVIO, J6 GIROUETTE, U1 ESP32-S3 Super Mini N4R2, U2 Module 3V3 Youmi

Commit message: Update 3D model and footprint for Regulator Module 3V3; add BOM documentation
- Modified the 3D shape of the Regulator Module 3V3 to adjust dimensions and colors.
- Updated the KiCad footprint for the Regulator Module 3V3, correcting pad positions and descriptions.
- Added a comprehensive Bill of Materials (BOM) for the MeteoHubSensor v1, detailing components, quantities, and specifications.
Connections:
- J1 pad 2: Net-(J1-Pin_2) -> GND
- J2 pad 2: GND -> /I2C_SCL
- J2 pad 3: /I2C_SCL -> /I2C_SDA
- J2 pad 4: /I2C_SDA -> GND
- U2 pad 3: Net-(U2-VOUT) -> +3V3
Routing:
- net GND: track 137.2 -> 0.00 mm, vias 5 -> 0
- net /VBAT: track 21.0 -> 23.5 mm
- net +3V3: track 119.1 -> 116.6 mm
- net /I2C_SDA: track 21.6 -> 19.1 mm
- net /I2C_SCL: track 16.5 -> 14.0 mm
Other:
- board text added: "DHT22"
- board text added: "GIROUETTE"
